Commit message: Add optional ground-truth 2D box camera to the simulation
Every COCO object in the house gets gz-sim's Label system (label = COCO
index). gt_boxes:=true adds a boundingbox_camera with the RGB camera's optics
and bridges its boxes to /oakd/gt_boxes (vision_msgs/Detection2DArray), for
detector evaluation.

Co-Authored-By: Claude Opus 5.5 <noreply@anthropic.com>

File: src/semantic_nav_bringup/urdf/oakd_semantic.urdf.xacro (robot description, xacro)
@@ -4,8 +4,10 @@
   urdf/sensors/oakd.urdf.xacro.
   Change for semantic_nav: image size, update rate and far clip are macro parameters
-  (upstream hard-codes 320x240 @ 30 Hz, far 100 m).
+  (upstream hard-codes 320x240 @ 30 Hz, far 100 m). gt_boxes:=true adds a
+  gz boundingbox_camera with identical optics that publishes ground-truth 2D
+  boxes of Label-ed models (detector evaluation only; costs one extra render pass).
 -->
 <robot xmlns:xacro="http://ros.org/wiki/xacro">
-<xacro:macro name="oakd_semantic" params="name:=oakd parent_link *origin model:=pro image_width:=640 image_height:=480 update_rate:=10 far_clip:=10.0">
+<xacro:macro name="oakd_semantic" params="name:=oakd parent_link *origin model:=pro image_width:=640 image_height:=480 update_rate:=10 far_clip:=10.0 gt_boxes:=false">
   <xacro:include filename="$(find irobot_create_description)/urdf/common_properties.urdf.xacro"/>
   <xacro:property name="mass"       value="0.061"/>
@@ -124,4 +126,26 @@
     <xacro:material_darkgray/>
   </gazebo>
+  <xacro:if value="${gt_boxes}">
+    <gazebo reference="${name}_rgb_camera_frame">
+      <sensor name="gt_boxes" type="boundingbox_camera">
+        <topic>${name}/gt_boxes</topic>
+        <camera>
+          <box_type>2d</box_type>
+          <horizontal_fov>1.25</horizontal_fov>
+          <image>
+            <width>${image_width}</width>
+            <height>${image_height}</height>
+          </image>
+          <clip>
+            <near>0.3</near>
+            <far>${far_clip}</far>
+          </clip>
+          <optical_frame_id>${name}_rgb_camera_optical_frame</optical_frame_id>
+        </camera>
+        <always_on>1</always_on>
+        <update_rate>${update_rate}</update_rate>
+      </sensor>
+    </gazebo>
+  </xacro:if>
   <gazebo reference="${name}_joint">
     <preserveFixedJoint>true</preserveFixedJoint>

File: src/semantic_nav_bringup/urdf/turtlebot4_semantic.urdf.xacro (robot description, xacro)
@@ -4,5 +4,5 @@
   urdf/standard/turtlebot4.urdf.xacro.
   Change for semantic_nav: includes oakd_semantic.urdf.xacro and exposes camera_width,
-  camera_height, camera_rate xacro args; uses rplidar_semantic.urdf.xacro
+  camera_height, camera_rate, gt_boxes xacro args; uses rplidar_semantic.urdf.xacro
   with a lidar_rate xacro arg.
 -->
@@ -12,4 +12,5 @@
   <xacro:arg name="camera_rate" default="10"/>
   <xacro:arg name="lidar_rate" default="10"/>
+  <xacro:arg name="gt_boxes" default="false"/>
   <!-- Base create3 model -->
   <xacro:include filename="$(find irobot_create_description)/urdf/create3.urdf.xacro" />
@@ -112,5 +113,5 @@
   <xacro:oakd_semantic model="pro" parent_link="oakd_camera_bracket"
                       image_width="$(arg camera_width)" image_height="$(arg camera_height)"
-                      update_rate="$(arg camera_rate)">
+                      update_rate="$(arg camera_rate)" gt_boxes="$(arg gt_boxes)">
     <origin xyz="${oakd_pro_x_offset} ${oakd_pro_y_offset} ${oakd_pro_z_offset}"/>
   </xacro:oakd_semantic>
